File: fuenteHack.kicad_pcb (KiCad board)
At the start: 2 copper layers, 45 x 29 mm, 18 parts, among them J1 USB_B_Micro, J2 Conn_01x02_Male, J3 Conn_01x02_Male, J4 Conn_01x02_Male, U1 LM1117-3.3, U2 TPS61087

Commit message: se realizan acabados para PCB
Parts:
- moved C1 31.8 mm to (145.2, 98.0), turned to 180 degrees
- moved C6 31.0 mm to (177.0, 99.0), turned to 180 degrees
- moved C3 28.5 mm to (147.8, 80.1), turned to 90 degrees
- moved C2 26.5 mm to (147.0, 89.0), turned to 270 degrees
- moved L1 20.9 mm to (171.8, 79.3)
- moved R2 11.5 mm to (162.1, 88.8), turned to 90 degrees
- moved C5 11.3 mm to (173.9, 88.5), turned to 270 degrees
- moved C4 10.0 mm to (163.5, 92.1)
- moved R3 8.69 mm to (166.1, 89.5), turned to 0 degrees
- moved D1 7.78 mm to (170.4, 92.9)
- moved 5V*J3 7.00 mm to (161.0, 79.1)
- moved R1 5.13 mm to (163.5, 85.3)
- moved U2 4.89 mm to (168.5, 86.3)
- moved U1 2.10 mm to (155.0, 89.0), turned to 180 degrees
- moved G*** 0.99 mm to (153.3, 98.3)
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- renumbered J4 to 12v*J4, J2 to 3.3V*J2, J3 to 5V*J3
Routing:
- net GND: track 0.00 -> 109.0 mm, vias 0 -> 2
- net +5V: track 0.00 -> 65.5 mm, vias 0 -> 2
- net +12V: track 0.00 -> 31.8 mm, vias 0 -> 2
- net +3V3: track 0.00 -> 26.7 mm, vias 0 -> 2
- net Net-(D1-Pad2): track 0.00 -> 19.3 mm, vias 0 -> 2
- net Net-(C4-Pad1): track 0.00 -> 9.16 mm
- net /FB: track 0.00 -> 8.42 mm
- net Net-(C5-Pad1): track 0.00 -> 7.33 mm, vias 0 -> 2
- net Net-(R1-Pad1): track 0.00 -> 3.90 mm
- added copper zone on B.Cu, net GND
- added copper zone on F.Cu, net GND
Other:
- rule trace_min: 0.2 -> 0.127
- rule via_min_drill: 0.3 -> 0.4
- rule via_min_size: 0.4 -> 0.5
