File: Proyecto_Final/Proyecto_Final.sch (KiCad schematic (older format))
At the start: 97 parts, among them J1 Conn_01x10, J10 Conn_01x02, J2 Conn_01x08, J3 USB_OTG, J4 Conn_01x08, J5 Conn_01x06, J6 Conn_01x02, J7 Conn_01x02, J8 Conn_02x03_Odd_Even, J9 Conn_02x03_Odd_Even, Q1 MMBT3904, Q2 MMBT3904, Q3 MMBT3904, Q4 MMBT3904, Q5 MMBT3904, Q6 MMBT3904, SW1 SW_Push, SW2 SW_Push, SW3 SW_Push, SW4 SW_Push, SW5 SW_Push, SW6 SW_Push, U1 TPS61087DSCR, U2 LM1117-3.3, U3 L293D, U4 FT232RL, U5 ATXMEGA32A4U-AU, U6 MODULE-BLUETOOTH-HC-05(34P-27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

Commit message: inicio del diseño PCB
Parts:
- C10, C3: footprint Capacitors_SMD:CP_Elec_4x4.5 -> Capacitor_SMD:CP_Elec_4x4.5
- C7: footprint Capacitors_SMD:CP_Elec_4x5.3 -> Capacitor_SMD:CP_Elec_4x5.3
- J1: footprint Pin_Headers:Pin_Header_Straight_1x10_Pitch2.54mm -> Connector_PinSocket_2.54mm:PinSocket_1x10_P2.54mm_Vertical
- J10: footprint Pin_Headers:Pin_Header_Straight_1x02_Pitch2.54mm -> Connector_PinHeader_2.54mm:PinHeader_1x02_P2.54mm_Vertical
- J2, J4: footprint Pin_Headers:Pin_Header_Straight_1x08_Pitch2.54mm -> Connector_PinSocket_2.54mm:PinSocket_1x08_P2.54mm_Vertical
- J5: footprint Pin_Headers:Pin_Header_Straight_1x06_Pitch2.54mm -> Connector_PinSocket_2.54mm:PinSocket_1x06_P2.54mm_Vertical
- J6, J7: footprint TerminalBlocks_Phoenix:TerminalBlock_Phoenix_MPT-2.54mm_2pol -> TerminalBlock_Phoenix:TerminalBlock_Phoenix_MPT-0,5-2-2.54_1x02_P2.54mm_Horizontal
- J8, J9: footprint Pin_Headers:Pin_Header_Straight_2x03_Pitch2.54mm -> Connector_PinSocket_2.54mm:PinSocket_2x03_P2.54mm_Vertical
- Q1, Q2, Q3, Q4, Q5, Q6: footprint TO_SOT_Packages_SMD:SOT-23_Handsoldering -> Package_TO_SOT_SMD:SOT-23
- R1, R10, R11, R12, R13, R14, R15, R16, R17, R18, R19, R2, R20, R21, R22, R23, R24, R25, R26, R27, R28, R29, R3, R30, R31, R32, R33, R34, R35, R36, R4, R5, R6, R7, R8, R9: footprint Resistors_SMD:R_1206_HandSoldering -> Resistor_SMD:R_1206_3216Metric
- RV1: footprint Potentiometers:Potentiometer_Trimmer_Bourns_PV36W -> Potentiometer_THT:Potentiometer_Bourns_3339P_Vertical
- SW1, SW2, SW3, SW4, SW5, SW6: footprint Buttons_Switches_SMD:SW_SPST_FSMSM -> Button_Switch_SMD:SW_SPST_FSMSM
- U2: footprint TO_SOT_Packages_SMD:TO-252-2 -> Package_TO_SOT_SMD:TO-252-2
- U5: footprint Housings_QFP:TQFP-44_10x10mm_Pitch0.8mm -> Package_QFP:TQFP-44_10x10mm_P0.8mm
- U6: footprint Platzi:HC-05 -> HC-05:BLUETOOTH-HC-05

Commit message: posicion inicial de componentes
Parts:
- D7: footprint LED_SMD:LED_RGB_Cree-PLCC-6_6x5mm_P2.1mm -> LED_THT:LED_D5.0mm-4_RGB_Wide_Pins
Changed lines of the file:
@@
 F 0 "D7" H 12200 2070 50  0000 C CNN
 F 1 "LED_RCGB" H 12200 1350 50  0000 C CNN
-F 2 "LED_SMD:LED_RGB_Cree-PLCC-6_6x5mm_P2.1mm" H 12200 1650 50  0001 C CNN
+F 2 "LED_THT:LED_D5.0mm-4_RGB_Wide_Pins" H 12200 1650 50  0001 C CNN
 F 3 "" H 12200 1650 50  0001 C CNN
 	1    12200 1700

Commit message: se crean zonas de tierra
Parts:
- RV1: footprint Potentiometer_THT:Potentiometer_Bourns_3339P_Vertical -> Potentiometer_THT:Potentiometer_Bourns_3296X_Horizontal
Changed lines of the file:
@@
 F 0 "RV1" V 6875 3700 50  0000 C CNN
 F 1 "R_POT_TRIM" V 6950 3700 50  0000 C CNN
-F 2 "Potentiometer_THT:Potentiometer_Bourns_3339P_Vertical" H 7050 3700 50  0001 C CNN
+F 2 "Potentiometer_THT:Potentiometer_Bourns_3296X_Horizontal" H 7050 3700 50  0001 C CNN
 F 3 "" H 7050 3700 50  0001 C CNN
 	1    7050 3700
